Commit message: urdf update

File: src/jawarm_description/urdf/jaw.urdf (robot description, URDF)
Before this commit: robot jawpixarm, 1 links, 0 joints
Links:
- added link baseToshoulder_link; visual mesh filename=package://jawarm_description/meshes/base_to_shoulder.STL scale=0.01 0.01 0.01
- added link p1_link
- added link p2_link
- added link servo1_link; visual mesh filename=package://jawarm_description/meshes/servo.STL scale=0.01 0.01 0.01
- added link servo2_link; visual mesh filename=package://jawarm_description/meshes/servo.STL scale=0.01 0.01 0.01
- added link servo3_link; visual mesh filename=package://jawarm_description/meshes/servo.STL scale=0.01 0.01 0.01
- added link shoulder_link; visual mesh filename=package://jawarm_description/meshes/shoulder.STL scale=0.01 0.01 0.01
- link base_link: geometry visual mesh filename=package://jawarm_description/meshes/base.STL scale=0.01 0.01 0.01
Joints:
- added joint baseToshoulder_to_p1: type revolute, parent p1_link, child baseToshoulder_link, origin xyz=0 0 0 rpy=0 0 0, axis 0 0 1, limit lower=-1.57 upper=1.57 effort=10 velocity=1.0
- added joint p1_to_servo1: type fixed, parent servo1_link, child p1_link, origin xyz=0.19 0.41 0.4 rpy=0 0 0
- added joint p2_to_servo2: type fixed, parent servo2_link, child p2_link, origin xyz=0.19 -0.001 0.155 rpy=0 1.5708 0
- added joint servo1_base: type fixed, parent base_link, child servo1_link, origin xyz=0 0 0 rpy=0 0 0
- added joint servo2_to_baseToshoulder: type fixed, parent baseToshoulder_link, child servo2_link, origin xyz=0 0 0 rpy=0 0 0
- added joint servo3_to_shoulder: type fixed, parent shoulder_link, child servo3_link, origin xyz=0 0 0 rpy=0 0 0
- added joint shoulder_to_p2: type revolute, parent p2_link, child shoulder_link, origin xyz=0 0 0 rpy=0 0 0, axis 0 0 1, limit lower=-1.57 upper=1.57 effort=10 velocity=1.0

Commit message: urdf update

File: src/jawarm_description/urdf/jaw.urdf (robot description, URDF)
Before this commit: robot jawpixarm, 8 links, 7 joints
Links:
- added link elbow_link; visual mesh filename=package://jawarm_description/meshes/elbow.STL scale=0.01 0.01 0.01
- added link p3_link
- added link p4_link
- added link servo4_link; visual mesh filename=package://jawarm_description/meshes/servo.STL scale=0.01 0.01 0.01
- added link wrist_link; visual mesh filename=package://jawarm_description/meshes/wrist.STL scale=0.01 0.01 0.01
Joints:
- added joint elbow_to_p3: type revolute, parent p3_link, child elbow_link, origin xyz=0 0 0 rpy=0 0 -1.5708, axis 0 0 1, limit lower=-1.57 upper=1.57 effort=10 velocity=1.0
- added joint p3_to_servo3: type fixed, parent servo3_link, child p3_link, origin xyz=-1.0 0.32 0 rpy=0 0 0
- added joint p4_to_servo4: type fixed, parent servo4_link, child p4_link, origin xyz=-1.0 1.589 0 rpy=0 0 0
- added joint servo4_to_elbow: type fixed, parent shoulder_link, child servo4_link, origin xyz=0 0 0 rpy=0 0 0
- added joint wrist_to_p4: type revolute, parent p4_link, child wrist_link, origin xyz=0 0 0 rpy=0 0 -1.5708, axis 0 0 1, limit lower=-1.57 upper=1.57 effort=10 velocity=1.0

Commit message: urdf update

File: src/jawarm_description/urdf/jaw.urdf (robot description, URDF)
Before this commit: robot jawpixarm, 13 links, 12 joints
Joints:
- joint p4_to_servo4: origin xyz=-1.0 1.589 0 rpy=0 0 0 -> xyz=-1.268 0.005 0 rpy=0 0 0
- joint servo4_to_elbow: parent shoulder_link -> elbow_link

Commit message: update urdf

File: src/jawarm_description/urdf/jaw.urdf (robot description, URDF)
Before this commit: robot jawpixarm, 13 links, 12 joints
Links:
- added link p5_link
- added link servo5_link; visual mesh filename=package://jawarm_description/meshes/servo.STL scale=0.01 0.01 0.01
- added link staticgrip_link; visual mesh filename=package://jawarm_description/meshes/static_gripper.STL scale=0.01 0.01 0.01
Joints:
- added joint p5_to_servo5: type fixed, parent servo5_link, child p5_link, origin xyz=0 0 0 rpy=0 1.5708 0
- added joint servo5_to_wrist: type fixed, parent wrist_link, child servo5_link, origin xyz=-0.141 -0.28 0 rpy=0 0 0
- added joint staticgrip_to_p5: type revolute, parent p5_link, child staticgrip_link, origin xyz=0.115 -0.38 0.139 rpy=1.5708 1.5708 0, axis 0 0 1, limit lower=-1.57 upper=1.57 effort=10 velocity=1.0

Commit message: update urdf

File: src/jawarm_description/urdf/jaw.urdf (robot description, URDF)
Before this commit: robot jawpixarm, 16 links, 15 joints
Links:
- added link mobilegrip_link; visual mesh filename=package://jawarm_description/meshes/mobile_gripper.STL scale=0.01 0.01 0.01
- added link p6_link
- added link servo6_link; visual mesh filename=package://jawarm_description/meshes/servo.STL scale=0.01 0.01 0.01
Joints:
- added joint mobilegrip_to_p6: type revolute, parent p6_link, child mobilegrip_link, origin xyz=0.335 -0.165 -0.17 rpy=3.1415 6.2831 1.5708, axis 0 1 0, limit lower=-1.57 upper=1.57 effort=10 velocity=1.0
- added joint p6_to_servo6: type fixed, parent servo6_link, child p6_link, origin xyz=0 0 0 rpy=3.1415 0 0
- added joint servo6_to_staticgrip: type fixed, parent staticgrip_link, child servo6_link, origin xyz=-0.141 -0.28 0 rpy=0 0 0

Commit message: update urdrf

File: src/jawarm_description/urdf/jaw.urdf (robot description, URDF)
Before this commit: robot jawpixarm, 19 links, 18 joints
Joints:
- joint mobilegrip_to_p6: origin xyz=0.335 -0.165 -0.17 rpy=3.1415 6.2831 1.5708 -> xyz=0.335 -0.165 -0.17 rpy=1.5708 6.2831 1.5708

Commit message: urdf updated

File: src/jawarm_description/urdf/jaw.urdf (robot description, URDF)
Before this commit: robot jawpixarm, 19 links, 18 joints
Links:
- link baseToshoulder_link: mass None -> 0.01; geometry collision mesh filename=package://jawarm_description/meshes/base_to_shoulder.STL scale=0.01 0.01 0.01; visual mesh filename=package://jawarm_description/meshes/base_to_shoulder.STL scale=0.01 0.01 0.01
- link base_link: mass None -> 0.02; geometry collision mesh filename=package://jawarm_description/meshes/base.STL scale=0.01 0.01 0.01; visual mesh filename=package://jawarm_description/meshes/base.STL scale=0.01 0.01 0.01
- link elbow_link: mass None -> 0.01; geometry collision mesh filename=package://jawarm_description/meshes/elbow.STL scale=0.01 0.01 0.01; visual mesh filename=package://jawarm_description/meshes/elbow.STL scale=0.01 0.01 0.01
- link mobilegrip_link: mass None -> 0.01; geometry collision mesh filename=package://jawarm_description/meshes/mobile_gripper.STL scale=0.01 0.01 0.01; visual mesh filename=package://jawarm_description/meshes/mobile_gripper.STL scale=0.01 0.01 0.01
- link servo1_link: mass None -> 0.0572; geometry collision mesh filename=package://jawarm_description/meshes/servo.STL scale=0.01 0.01 0.01; visual mesh filename=package://jawarm_description/meshes/servo.STL scale=0.01 0.01 0.01
- link servo2_link: mass None -> 0.0572; geometry collision mesh filename=package://jawarm_description/meshes/servo.STL scale=0.01 0.01 0.01; visual mesh filename=package://jawarm_description/meshes/servo.STL scale=0.01 0.01 0.01
- link servo3_link: mass None -> 0.0572; geometry collision mesh filename=package://jawarm_description/meshes/servo.STL scale=0.01 0.01 0.01; visual mesh filename=package://jawarm_description/meshes/servo.STL scale=0.01 0.01 0.01
- link servo4_link: mass None -> 0.0572; geometry collision mesh filename=package://jawarm_description/meshes/servo.STL scale=0.01 0.01 0.01; visual mesh filename=package://jawarm_description/meshes/servo.STL scale=0.01 0.01 0.01
- link servo5_link: mass None -> 0.0572; geometry collision mesh filename=package://jawarm_description/meshes/servo.STL scale=0.01 0.01 0.01; visual mesh filename=package://jawarm_description/meshes/servo.STL scale=0.01 0.01 0.01
- link servo6_link: mass None -> 0.0572; geometry collision mesh filename=package://jawarm_description/meshes/servo.STL scale=0.01 0.01 0.01; visual mesh filename=package://jawarm_description/meshes/servo.STL scale=0.01 0.01 0.01
- link shoulder_link: mass None -> 0.01; geometry collision mesh filename=package://jawarm_description/meshes/shoulder.STL scale=0.01 0.01 0.01; visual mesh filename=package://jawarm_description/meshes/shoulder.STL scale=0.01 0.01 0.01
- link staticgrip_link: mass None -> 0.01; geometry collision mesh filename=package://jawarm_description/meshes/static_gripper.STL scale=0.01 0.01 0.01; visual mesh filename=package://jawarm_description/meshes/static_gripper.STL scale=0.01 0.01 0.01
- link wrist_link: mass None -> 0.01; geometry collision mesh filename=package://jawarm_description/meshes/wrist.STL scale=0.01 0.01 0.01; visual mesh filename=package://jawarm_description/meshes/wrist.STL scale=0.01 0.01 0.01
Joints:
- joint mobilegrip_to_p6: axis 0 1 0 -> 0 0 1
