Commit message: uploaded the last version of STL files

File: my_robot_description/urdf/mobile_base.xacro (robot description, xacro)
@@ -3,16 +3,23 @@
     <xacro:include filename="common_properties.xacro" />
     <xacro:property name="m_scale" value="0.01 0.01 0.01" />
+    <xacro:macro name="default_inertial" params="mass">
+        <inertial>
+            <origin xyz="0 0 0" rpy="0 0 0"/>
+            <mass value="${mass}"/>
+            <inertia ixx="1.0e-04" iyy="1.0e-04" izz="1.0e-04" ixy="0.0" ixz="0.0" iyz="0.0"/>
+        </inertial>
+    </xacro:macro>
     <link name="base_link">
         <visual>
-            <origin xyz="-1.05 1.5 0" rpy="${pi / 2.0} 0 0"/>
-            <geometry><mesh filename="package://my_robot_description/meshes/base.STL" scale="${m_scale}"/></geometry>
-            <material name="blue" />
-        </visual>
-        <collision>
-            <origin xyz="-1.05 1.5 0" rpy="${pi / 2.0} 0 0"/>
-            <geometry><mesh filename="package://my_robot_description/meshes/base.STL" scale="${m_scale}"/></geometry>
+            <origin xyz="-0.52 0.8 0" rpy="${pi / 2.0} 0 0"/>
+            <geometry><mesh filename="package://my_robot_description/meshes/baza.STL" scale="${m_scale}"/></geometry>
+            <material name="blue" />
+        </visual>
+        <collision>
+            <origin xyz="-0.52 0.8 0" rpy="${pi / 2.0} 0 0"/>
+            <geometry><mesh filename="package://my_robot_description/meshes/baza.STL" scale="${m_scale}"/></geometry>
         </collision>
         <inertial>
-            <origin xyz="-1.05 1.5 0" rpy="0 0 0"/><mass value="0.02"/>
+            <origin xyz="-0.52 0.8 0" rpy="0 0 0"/><mass value="0.02"/>
             <inertia ixx="1.04e-04" iyy="1.04e-04" izz="2.08e-04" ixy="0.0" ixz="0.0" iyz="0.0"/>
         </inertial>
@@ -20,8 +27,12 @@
     <link name="servo1_link">
         <visual>
-            <origin xyz="0.05 0.52 0.03" rpy="${pi / 2.0} 0 0"/>
-            <geometry><mesh filename="package://my_robot_description/meshes/servo.STL" scale="${m_scale}"/></geometry>
-            <material name="blue" />
-        </visual>
+            <origin xyz="0.05 0.52 0.278" rpy="${pi / 2.0} 0 0"/>
+            <geometry><mesh filename="package://my_robot_description/meshes/servo.STL" scale="${m_scale}"/></geometry>
+            <material name="blue" />
+        </visual>
+        <collision>
+            <origin xyz="0.05 0.52 0.278" rpy="${pi / 2.0} 0 0"/>
+            <geometry><mesh filename="package://my_robot_description/meshes/servo.STL" scale="${m_scale}"/></geometry>
+        </collision>
         <xacro:servo_inertial />
     </link>
@@ -35,8 +46,13 @@
     <link name="baseToshoulder_link">
         <visual>
-            <origin xyz="-0.2 -0.388 -0.2" rpy="0 0 0"/>
+            <origin xyz="0.265 0.52 -0.23" rpy="${pi * 1.5} ${-pi} ${pi / 2.0}"/>
             <geometry><mesh filename="package://my_robot_description/meshes/base_to_shoulder.STL" scale="${m_scale}"/></geometry>
             <material name="blue" />
         </visual>
+        <collision>
+            <origin xyz="0.265 0.52 -0.23" rpy="${pi * 1.5} ${-pi} ${pi / 2.0}"/>
+            <geometry><mesh filename="package://my_robot_description/meshes/base_to_shoulder.STL" scale="${m_scale}"/></geometry>
+        </collision>
+        <xacro:default_inertial mass="0.02"/>
     </link>
     <joint name="joint1" type="revolute">
@@ -46,8 +62,12 @@
     <link name="servo2_link">
         <visual>
+            <origin xyz="0.165 0.49 0.85" rpy="0 ${pi} ${pi / 2.0}"/>
+            <geometry><mesh filename="package://my_robot_description/meshes/servo.STL" scale="${m_scale}"/></geometry>
+            <material name="blue" />
+        </visual>
+        <collision>
             <origin xyz="-0.17 0.109 0.3" rpy="${pi / 2.0} ${pi / 2.0} 0"/>
             <geometry><mesh filename="package://my_robot_description/meshes/servo.STL" scale="${m_scale}"/></geometry>
-            <material name="blue" />
-        </visual>
+        </collision>
         <xacro:servo_inertial />
     </link>
@@ -55,13 +75,19 @@
         <parent link="baseToshoulder_link"/><child link="servo2_link"/>
     </joint>
-    <link name="p2_link"/><link name="shoulder_link">
-        <visual>
-            <origin xyz="0.11 0.157 0.03" rpy="0 ${pi / 2.0} ${pi}"/>
+    <link name="p2_link"/>
+    <link name="shoulder_link">
+        <visual>
+            <origin xyz="0.11 0.157 0.1" rpy="0 ${pi / 2.0} ${pi}"/>
             <geometry><mesh filename="package://my_robot_description/meshes/shoulder.STL" scale="${m_scale}"/></geometry>
             <material name="blue" />
         </visual>
+        <collision>
+            <origin xyz="0.11 0.157 0.1" rpy="0 ${pi / 2.0} ${pi}"/>
+            <geometry><mesh filename="package://my_robot_description/meshes/shoulder.STL" scale="${m_scale}"/></geometry>
+        </collision>
+        <xacro:default_inertial mass="0.02"/>
     </link>
     <joint name="p2_to_servo2" type="fixed">
-        <origin xyz="0.19 -0.001 0.155" rpy="0 ${pi / 2.0} 0"/><parent link="servo2_link"/><child link="p2_link"/>
+        <origin xyz="0.19 0.347 0.74" rpy="0 ${pi / 2.0} 0"/><parent link="servo2_link"/><child link="p2_link"/>
     </joint>
     <joint name="joint2" type="revolute">
@@ -75,4 +101,8 @@
             <material name="blue" />
         </visual>
+        <collision>
+            <origin xyz="-1.139 0.431 -0.36" rpy="-${pi / 2.0} ${pi} ${pi}"/>
+            <geometry><mesh filename="package://my_robot_description/meshes/servo.STL" scale="${m_scale}"/></geometry>
+        </collision>
         <xacro:servo_inertial />
     </link>
@@ -80,5 +110,6 @@
         <parent link="shoulder_link"/><child link="servo3_link"/>
     </joint>
-    <link name="p3_link"/><link name="elbow_link">
+    <link name="p3_link"/>
+    <link name="elbow_link">
         <visual>
             <origin xyz="0.113 0.148 0.03" rpy="0 ${pi / 2.0} ${pi}"/>
@@ -86,4 +117,9 @@
             <material name="blue" />
         </visual>
+        <collision>
+            <origin xyz="0.113 0.148 0.03" rpy="0 ${pi / 2.0} ${pi}"/>
+            <geometry><mesh filename="package://my_robot_description/meshes/elbow.STL" scale="${m_scale}"/></geometry>
+        </collision>
+        <xacro:default_inertial mass="0.02"/>
     </link>
     <joint name="p3_to_servo3" type="fixed">
@@ -100,4 +136,8 @@
             <material name="blue" />
         </visual>
+        <collision>
+            <origin xyz="-1.38 -0.139 -0.36" rpy="${pi / 2.0} 0 ${pi / 2.0}"/>
+            <geometry><mesh filename="package://my_robot_description/meshes/servo.STL" scale="${m_scale}"/></geometry>
+        </collision>
         <xacro:servo_inertial />
     </link>
@@ -105,5 +145,6 @@
         <parent link="elbow_link"/><child link="servo4_link"/>
     </joint>
-    <link name="p4_link"/><link name="wrist_link">
+    <link name="p4_link"/>
+    <link name="wrist_link">
         <visual>
             <origin xyz="0.1429 -0.2877 0.03" rpy="${pi / 2.0} ${pi / 2.0} ${pi}"/>
@@ -111,4 +152,9 @@
             <material name="blue" />
         </visual>
+        <collision>
+            <origin xyz="0.1429 -0.2877 0.03" rpy="${pi / 2.0} ${pi / 2.0} ${pi}"/>
+            <geometry><mesh filename="package://my_robot_description/meshes/wrist.STL" scale="${m_scale}"/></geometry>
+        </collision>
+        <xacro:default_inertial mass="0.02"/>
     </link>
     <joint name="p4_to_servo4" type="fixed">
@@ -125,4 +171,8 @@
             <material name="blue" />
         </visual>
+        <collision>
+            <origin xyz="0 -0.01 0" rpy="${pi} 0 0"/>
+            <geometry><mesh filename="package://my_robot_description/meshes/servo.STL" scale="${m_scale}"/></geometry>
+        </collision>
         <xacro:servo_inertial />
     </link>
@@ -130,5 +180,6 @@
         <origin xyz="-0.141 -0.28 0" rpy="0 0 0"/><parent link="wrist_link"/><child link="servo5_link"/>
     </joint>
-    <link name="p5_link"/><link name="staticgrip_link">
+    <link name="p5_link"/>
+    <link name="staticgrip_link">
         <visual>
             <origin xyz="0.2 0.335 0" rpy="${pi / 2.0} 0 4.7123"/>
@@ -136,4 +187,9 @@
             <material name="blue" />
         </visual>
+        <collision>
+            <origin xyz="0.2 0.335 0" rpy="${pi / 2.0} 0 4.7123"/>
+            <geometry><mesh filename="package://my_robot_description/meshes/static_gripper.STL" scale="${m_scale}"/></geometry>
+        </collision>
+        <xacro:default_inertial mass="0.01"/>
     </link>
     <joint name="p5_to_servo5" type="fixed">
@@ -150,4 +206,8 @@
             <material name="blue" />
         </visual>
+        <collision>
+            <origin xyz="-0.0325 0.05 0.03" rpy="${pi / 2.0} -${pi / 2.0} ${pi}"/>
+            <geometry><mesh filename="package://my_robot_description/meshes/servo.STL" scale="${m_scale}"/></geometry>
+        </collision>
         <xacro:servo_inertial />
     </link>
@@ -155,5 +215,6 @@
         <origin xyz="-0.141 -0.28 0" rpy="0 0 0"/><parent link="staticgrip_link"/><child link="servo6_link"/>
     </joint>
-    <link name="p6_link"/><link name="mobilegrip_link">
+    <link name="p6_link"/>
+    <link name="mobilegrip_link">
         <visual>
             <origin xyz="0.1125 0.13 -0.415" rpy="0 0 ${pi}"/>
@@ -161,4 +222,9 @@
             <material name="blue" />
         </visual>
+        <collision>
+            <origin xyz="0.1125 0.13 -0.415" rpy="0 0 ${pi}"/>
+            <geometry><mesh filename="package://my_robot_description/meshes/mobile_gripper.STL" scale="${m_scale}"/></geometry>
+        </collision>
+        <xacro:default_inertial mass="0.01"/>
     </link>
     <joint name="p6_to_servo6" type="fixed">

Commit message: update

File: my_robot_description/urdf/mobile_base.xacro (robot description, xacro)
@@ -40,5 +40,7 @@
         <parent link="base_link"/><child link="servo1_link"/><origin xyz="0 0 0" rpy="0 0 0"/>
     </joint>
-    <link name="p1_link"/>
+    <link name="p1_link">
+        <collision><geometry><sphere radius="0.0001"/></geometry></collision>
+    </link>
     <joint name="p1_to_servo1" type="fixed">
         <origin xyz="0.19 0.41 0.4" rpy="0 0 0"/><parent link="servo1_link"/><child link="p1_link"/>
@@ -67,5 +69,5 @@
         </visual>
         <collision>
-            <origin xyz="-0.17 0.109 0.3" rpy="${pi / 2.0} ${pi / 2.0} 0"/>
+            <origin xyz="0.165 0.49 0.85" rpy="0 ${pi} ${pi / 2.0}"/>
             <geometry><mesh filename="package://my_robot_description/meshes/servo.STL" scale="${m_scale}"/></geometry>
         </collision>
@@ -75,5 +77,7 @@
         <parent link="baseToshoulder_link"/><child link="servo2_link"/>
     </joint>
-    <link name="p2_link"/>
+    <link name="p2_link">
+        <collision><geometry><sphere radius="0.0001"/></geometry></collision>
+    </link>
     <link name="shoulder_link">
         <visual>
@@ -110,5 +114,7 @@
         <parent link="shoulder_link"/><child link="servo3_link"/>
     </joint>
-    <link name="p3_link"/>
+    <link name="p3_link">
+        <collision><geometry><sphere radius="0.0001"/></geometry></collision>
+    </link>
     <link name="elbow_link">
         <visual>
@@ -145,5 +151,7 @@
         <parent link="elbow_link"/><child link="servo4_link"/>
     </joint>
-    <link name="p4_link"/>
+    <link name="p4_link">
+        <collision><geometry><sphere radius="0.0001"/></geometry></collision>
+    </link>
     <link name="wrist_link">
         <visual>
@@ -180,5 +188,7 @@
         <origin xyz="-0.141 -0.28 0" rpy="0 0 0"/><parent link="wrist_link"/><child link="servo5_link"/>
     </joint>
-    <link name="p5_link"/>
+    <link name="p5_link">
+        <collision><geometry><sphere radius="0.0001"/></geometry></collision>
+    </link>
     <link name="staticgrip_link">
         <visual>
@@ -215,5 +225,7 @@
         <origin xyz="-0.141 -0.28 0" rpy="0 0 0"/><parent link="staticgrip_link"/><child link="servo6_link"/>
     </joint>
-    <link name="p6_link"/>
+    <link name="p6_link">
+        <collision><geometry><sphere radius="0.0001"/></geometry></collision>
+    </link>
     <link name="mobilegrip_link">
         <visual>

File: my_robot_description/urdf/my_robot.urdf.xacro (robot description, xacro)
@@ -2,4 +2,3 @@
 <robot name="my_robot" xmlns:xacro="http://www.ros.org/wiki/xacro">
     <xacro:include filename="mobile_base.xacro" />
-    <xacro:include filename="mobile_base.ros2_control.xacro" />
 </robot>
