Commit message: modified stls

File: my_robot_description/urdf/mobile_base.xacro (robot description, xacro)
@@ -82,10 +82,10 @@
     <link name="shoulder_link">
         <visual>
-            <origin xyz="0.11 0.157 0.1" rpy="0 ${pi / 2.0} ${pi}"/>
+            <origin xyz="0.136 0.15 0.07" rpy="0 ${pi / 2.0} ${pi}"/>
             <geometry><mesh filename="package://my_robot_description/meshes/shoulder.STL" scale="${m_scale}"/></geometry>
             <material name="blue" />
         </visual>
         <collision>
-            <origin xyz="0.11 0.157 0.1" rpy="0 ${pi / 2.0} ${pi}"/>
+            <origin xyz="0.136 0.15 0.07" rpy="0 ${pi / 2.0} ${pi}"/>
             <geometry><mesh filename="package://my_robot_description/meshes/shoulder.STL" scale="${m_scale}"/></geometry>
         </collision>
@@ -101,10 +101,10 @@
     <link name="servo3_link">
         <visual>
-            <origin xyz="-1.139 0.431 -0.36" rpy="-${pi / 2.0} ${pi} ${pi}"/>
-            <geometry><mesh filename="package://my_robot_description/meshes/servo.STL" scale="${m_scale}"/></geometry>
-            <material name="blue" />
-        </visual>
-        <collision>
-            <origin xyz="-1.139 0.431 -0.36" rpy="-${pi / 2.0} ${pi} ${pi}"/>
+            <origin xyz="-0.904 0.437 -0.363" rpy="-${pi / 2.0} ${pi} ${pi}"/>
+            <geometry><mesh filename="package://my_robot_description/meshes/servo.STL" scale="${m_scale}"/></geometry>
+            <material name="blue" />
+        </visual>
+        <collision>
+            <origin xyz="-0.904 0.437 -0.363" rpy="-${pi / 2.0} ${pi} ${pi}"/>
             <geometry><mesh filename="package://my_robot_description/meshes/servo.STL" scale="${m_scale}"/></geometry>
         </collision>
@@ -130,5 +130,5 @@
     </link>
     <joint name="p3_to_servo3" type="fixed">
-        <origin xyz="-1.0 0.32 0" rpy="0 0 0"/><parent link="servo3_link"/><child link="p3_link"/>
+        <origin xyz="-0.768 0.325 0" rpy="0 0 0"/><parent link="servo3_link"/><child link="p3_link"/>
     </joint>
     <joint name="joint3" type="revolute">
@@ -138,10 +138,10 @@
     <link name="servo4_link">
         <visual>
-            <origin xyz="-1.38 -0.139 -0.36" rpy="${pi / 2.0} 0 ${pi / 2.0}"/>
-            <geometry><mesh filename="package://my_robot_description/meshes/servo.STL" scale="${m_scale}"/></geometry>
-            <material name="blue" />
-        </visual>
-        <collision>
-            <origin xyz="-1.38 -0.139 -0.36" rpy="${pi / 2.0} 0 ${pi / 2.0}"/>
+            <origin xyz="-1.131 -0.139 -0.36" rpy="${pi / 2.0} 0 ${pi / 2.0}"/>
+            <geometry><mesh filename="package://my_robot_description/meshes/servo.STL" scale="${m_scale}"/></geometry>
+            <material name="blue" />
+        </visual>
+        <collision>
+            <origin xyz="-1.131 -0.139 -0.36" rpy="${pi / 2.0} 0 ${pi / 2.0}"/>
             <geometry><mesh filename="package://my_robot_description/meshes/servo.STL" scale="${m_scale}"/></geometry>
         </collision>
@@ -167,5 +167,5 @@
     </link>
     <joint name="p4_to_servo4" type="fixed">
-        <origin xyz="-1.268 0.005 0" rpy="0 0 0"/><parent link="servo4_link"/><child link="p4_link"/>
+        <origin xyz="-1.0185 0.005 0" rpy="0 0 0"/><parent link="servo4_link"/><child link="p4_link"/>
     </joint>
     <joint name="joint4" type="revolute">

Commit message: updates

File: my_robot_description/urdf/mobile_base.xacro (robot description, xacro)
@@ -2,19 +2,9 @@
 <robot xmlns:xacro="http://www.ros.org/wiki/xacro">
     <xacro:include filename="common_properties.xacro" />
-    <!-- ===================== units and physical constants =====================
-         All lengths are metres, all angles radians.
-         STL files are exported from CAD in millimetres, so m_scale = 0.001. -->
     <xacro:property name="m_scale" value="0.001 0.001 0.001" />
-    <!-- XL430-W250-T: stall torque about 1.5 N.m at 12 V, no-load speed about 57 rpm (6.0 rad/s).
-         Check both against the ROBOTIS e-manual. These are URDF limits, not driver settings. -->
     <xacro:property name="servo_effort" value="1.5" />
     <xacro:property name="servo_velocity" value="4.0" />
     <xacro:property name="servo_mass" value="0.0572" />
-    <!-- Effective density of the 3D-printed parts [kg/m^3]. Solid PLA is 1240; with walls + infill
-         a printed part is typically 40-60 % of that. Weigh a part and adjust: every printed link's
-         mass and inertia follow from (this density x the STL volume). -->
     <xacro:property name="print_density" value="620" />
-    <!-- Gripper (joint6). q = 0: moving jaw at 90 deg to the fixed jaw (open).
-         In the CAD model the fingers touch at -1.84 rad; -1.90 lets the current-limited servo squeeze. -->
     <xacro:property name="gripper_closed" value="-1.90" />
     <xacro:property name="gripper_open_max" value="0.30" />
@@ -30,6 +20,4 @@
         </collision>
     </link>
-    <!-- Desk surface. Collision only (invisible), top 0.5 mm below the base so it never touches the arm at rest.
-         Without it MoveIt can plan joint2 > ~+0.65 rad or joint3 < ~-0.85 rad, which drives the arm into the desk. -->
     <link name="table_link">
         <collision>
@@ -130,13 +118,13 @@
     <link name="elbow_link">
         <visual>
-            <origin xyz="0.0113 0.0148 0.003" rpy="0 ${pi / 2.0} ${pi}"/>
+            <origin xyz="0.011154 -0.01491 -0.0395" rpy="-0.009818 -${pi / 2.0} 0"/>
             <geometry><mesh filename="package://my_robot_description/meshes/elbow.STL" scale="${m_scale}"/></geometry>
             <material name="blue" />
         </visual>
         <collision>
-            <origin xyz="0.0113 0.0148 0.003" rpy="0 ${pi / 2.0} ${pi}"/>
+            <origin xyz="0.011154 -0.01491 -0.0395" rpy="-0.009818 -${pi / 2.0} 0"/>
             <geometry><mesh filename="package://my_robot_description/meshes/elbow.STL" scale="${m_scale}"/></geometry>
         </collision>
-        <xacro:mesh_inertial mass="${print_density * 3.1474e-05}" xyz="-0.040343 0.000661 -0.018793" ixx="2.8653e-04" iyy="5.6628e-04" izz="4.7095e-04" ixy="-1.7047e-06" ixz="7.6556e-06" iyz="2.6038e-08"/>
+        <xacro:mesh_inertial mass="${print_density * 3.1474e-05}" xyz="-0.040347 -0.000265 -0.017707" ixx="2.8659e-04" iyy="5.6622e-04" izz="4.7095e-04" ixy="4.4509e-06" ixz="-7.6550e-06" iyz="1.0120e-07"/>
     </link>
     <joint name="p3_to_servo3" type="fixed">
@@ -160,5 +148,5 @@
     </link>
     <joint name="servo4_to_elbow" type="fixed">
-        <parent link="elbow_link"/><child link="servo4_link"/>
+        <origin xyz="0 0 -0.0365" rpy="${pi} 0 -0.009818"/><parent link="elbow_link"/><child link="servo4_link"/>
     </joint>
     <link name="p4_link"/>

Commit message: updates

File: my_robot_description/urdf/mobile_base.xacro (robot description, xacro)
@@ -205,4 +205,9 @@
         <axis xyz="0 0 1"/><limit effort="${servo_effort}" velocity="${servo_velocity}" lower="-${pi / 2.0}" upper="${pi / 2.0}"/>
     </joint>
+    <link name="tcp_link"/>
+    <joint name="staticgrip_to_tcp" type="fixed">
+        <parent link="staticgrip_link"/><child link="tcp_link"/>
+        <origin xyz="-0.0002 0.0161 0.0849" rpy="${pi} -${pi / 2.0} 0"/>
+    </joint>
     <link name="servo6_link">
         <visual>

File: my_robot_description/urdf/my_robot.ros2_control.xacro (robot description, xacro)
@@ -12,4 +12,5 @@
               <param name="serial_port">/dev/ttyUSB0</param>
               <param name="baud_rate">1000000</param>
+              <!--<param name="calibrate_on_start">false</param>-->
             </hardware>
             <joint name="joint1">
