Commit message: update

File: my_robot_description/urdf/mobile_base.ros2_control.xacro (robot description, xacro)
@@ -3,7 +3,7 @@
     <ros2_control name="MobileBaseHardwareInterface" type="system">
         <hardware>
-          <!-- <plugin>mock_components/GenericSystem</plugin>
-            <param name="calculate_dynamics">true</param> -->
             <plugin>mobile_base_hardware/MobileBaseHardwareInterface</plugin>
+            <param name="serial_port">/dev/ttyUSB0</param>
+            <param name="baud_rate">1000000</param>
         </hardware>
         <joint name="joint1">

File: my_robot_description/urdf/mobile_base.xacro (robot description, xacro)
@@ -245,5 +245,5 @@
     <joint name="joint6" type="revolute">
         <origin xyz="0.335 -0.165 -0.17" rpy="${pi / 2.0} 6.2831 ${pi / 2.0}"/><parent link="p6_link"/><child link="mobilegrip_link"/>
-        <axis xyz="0 0 1"/><limit effort="10" velocity="1.0" lower="-${pi / 2.0}" upper="${pi / 2.0}"/>
+        <axis xyz="0 0 1"/><limit effort="10" velocity="1.0" lower="-${pi}" upper="${pi}"/>
     </joint>
 </robot>

File: my_robot_description/urdf/my_robot.urdf.xacro (robot description, xacro)
@@ -1,4 +1,7 @@
 <?xml version="1.0"?>
 <robot name="my_robot" xmlns:xacro="http://www.ros.org/wiki/xacro">
-    <xacro:include filename="mobile_base.xacro" />
+    <xacro:arg name="initial_positions_file" default="$(find my_robot_description)/config/initial_positions.yaml"/>
+    <xacro:include filename="$(find my_robot_description)/urdf/mobile_base.xacro" />
+    <xacro:include filename="$(find my_robot_description)/urdf/my_robot.ros2_control.xacro" />
+    <xacro:my_robot_ros2_control name="ArmSystem" initial_positions_file="$(arg initial_positions_file)"/>
 </robot>

File: my_robot_moveit_config/config/my_robot.urdf.xacro (robot description, xacro)
@@ -1,9 +1,7 @@
 <?xml version="1.0"?>
-<robot xmlns:xacro="http://www.ros.org/wiki/xacro" name="my_robot">
-    <xacro:arg name="initial_positions_file" default="initial_positions.yaml" />
-    <!-- Import my_robot urdf file -->
-    <xacro:include filename="$(find my_robot_description)/urdf/my_robot.urdf.xacro" />
-    <!-- Import control_xacro -->
-    <xacro:include filename="my_robot.ros2_control.xacro" />
+<robot name="my_robot" xmlns:xacro="http://www.ros.org/wiki/xacro">
+    <xacro:arg name="initial_positions_file" default="$(find my_robot_description)/config/initial_positions.yaml"/>
+    <xacro:include filename="$(find my_robot_description)/urdf/mobile_base.xacro" />
+    <xacro:include filename="$(find my_robot_description)/urdf/my_robot.ros2_control.xacro" />
     <xacro:my_robot_ros2_control name="FakeSystem" initial_positions_file="$(arg initial_positions_file)"/>
 </robot>
