Commit message: latest updates

File: my_robot_description/urdf/jaw.urdf (robot description, URDF)
Before this commit: robot jaw_roboarm, 19 links, 18 joints
Joints:
- joint joint1: limit lower=-1.57079632679 upper=1.57079632679 effort=10 velocity=1.0 -> lower=-1.5708 upper=1.5708 effort=10 velocity=1.0
- joint joint2: axis 0 0 1 -> 0 0 -1; limit lower=-1.57079632679 upper=1.57079632679 effort=10 velocity=1.0 -> lower=-1.5708 upper=1.5708 effort=10 velocity=1.0
- joint joint3: limit lower=-1.57079632679 upper=1.57079632679 effort=10 velocity=1.0 -> lower=-1.5708 upper=1.5708 effort=10 velocity=1.0
- joint joint4: limit lower=-1.57079632679 upper=1.57079632679 effort=10 velocity=1.0 -> lower=-1.5708 upper=1.5708 effort=10 velocity=1.0
- joint joint5: limit lower=-1.57079632679 upper=1.57079632679 effort=10 velocity=1.0 -> lower=-1.5708 upper=1.5708 effort=10 velocity=1.0; origin xyz=0.115 -0.38 0.139 rpy=1.57079632679 1.57079632679 0 -> xyz=0.115 -0.38 0.139 rpy=1.5708 1.5708 0
- joint joint6: limit lower=-1.57079632679 upper=1.57079632679 effort=10 velocity=1.0 -> lower=-1.5708 upper=1.5708 effort=10 velocity=1.0; origin xyz=0.335 -0.165 -0.17 rpy=1.57079632679 6.2831 1.57079632679 -> xyz=0.335 -0.165 -0.17 rpy=1.5708 0 1.5708
- joint p2_to_servo2: origin xyz=0.19 0.347 0.74 rpy=0 1.57079632679 0 -> xyz=0.19 0.347 0.74 rpy=0 1.5708 0
- joint p5_to_servo5: origin xyz=0 0 0 rpy=0 1.57079632679 0 -> xyz=0 0 0 rpy=0 1.5708 0
- joint p6_to_servo6: origin xyz=0 0 0 rpy=3.14159265359 0 0 -> xyz=0 0 0 rpy=3.1416 0 0

File: my_robot_description/urdf/mobile_base.xacro (robot description, xacro)
@@ -96,5 +96,5 @@
     </joint>
     <joint name="joint2" type="revolute">
-        <parent link="p2_link"/><child link="shoulder_link"/><axis xyz="0 0 1"/>
+        <parent link="p2_link"/><child link="shoulder_link"/><axis xyz="0 0 -1"/>
         <limit effort="10" velocity="1.0" lower="-${pi / 2.0}" upper="${pi / 2.0}"/>
     </joint>
@@ -230,10 +230,10 @@
     <link name="mobilegrip_link">
         <visual>
-            <origin xyz="0.1125 0.13 -0.415" rpy="0 0 ${pi}"/>
+            <origin xyz="-0.12 0.1 -0.415" rpy="0 0 -${pi / 2}"/>
             <geometry><mesh filename="package://my_robot_description/meshes/mobile_gripper.STL" scale="${m_scale}"/></geometry>
             <material name="blue" />
         </visual>
         <collision>
-            <origin xyz="0.1125 0.13 -0.415" rpy="0 0 ${pi}"/>
+            <origin xyz="-0.12 0.1 -0.415" rpy="0 0 -${pi / 2}"/>
             <geometry><mesh filename="package://my_robot_description/meshes/mobile_gripper.STL" scale="${m_scale}"/></geometry>
         </collision>
@@ -245,5 +245,5 @@
     <joint name="joint6" type="revolute">
         <origin xyz="0.335 -0.165 -0.17" rpy="${pi / 2.0} 6.2831 ${pi / 2.0}"/><parent link="p6_link"/><child link="mobilegrip_link"/>
-        <axis xyz="0 0 1"/><limit effort="10" velocity="1.0" lower="-${pi}" upper="${pi}"/>
+        <axis xyz="0 0 1"/><limit effort="10" velocity="1.0" lower="-${pi / 2}" upper="${pi / 2}"/>
     </joint>
 </robot>
