Commit message: updates

File: my_robot_description/urdf/common_properties.xacro (robot description, xacro)
@@ -4,9 +4,14 @@
         <color rgba="0.2 0.2 0.8 1"/>
     </material>
-    <xacro:macro name="servo_inertial">
+    <!-- Inertial computed from the link's mesh (uniform density):
+         xyz          = centre of mass in the link frame [m]
+         ixx ... iyz  = inertia about the centre of mass, PER KILOGRAM, in link axes [m^2]
+         mass         = kg; the tensor is multiplied by it, so changing the mass keeps the geometry right -->
+    <xacro:macro name="mesh_inertial" params="mass xyz ixx iyy izz ixy ixz iyz">
         <inertial>
-            <origin xyz="0.05 0.52 0.03" rpy="${pi / 2.0} 0 0"/>
-            <mass value="0.0572"/>
-            <inertia ixx="6.2e-05" iyy="7.8e-05" izz="1.0e-04" ixy="0.0" ixz="0.0" iyz="0.0"/>
+            <origin xyz="${xyz}" rpy="0 0 0"/>
+            <mass value="${mass}"/>
+            <inertia ixx="${mass * ixx}" iyy="${mass * iyy}" izz="${mass * izz}"
+                     ixy="${mass * ixy}" ixz="${mass * ixz}" iyz="${mass * iyz}"/>
         </inertial>
     </xacro:macro>
